File: pcb/interconnects.kicad_sch (KiCad schematic)
At the start: 0 parts

Commit message: Bake everything into the PCB (+ commit the intermediates)
This is mostly for traceability reproducibility reasons.
In practice, the best way to bake a different design would be to branch
off just before this commit
Other:
- note added: "$abc$2582$auto$alumacc.cc:512:replace_alu$174.CO[2]_new"
- note added: "$abc$2582$auto$alumacc.cc:512:replace_alu$174.CO[4]_new"
- note added: "$abc$2582$auto$alumacc.cc:512:replace_alu$174.CO[6]_new"
- note added: "$abc$2582$auto$alumacc.cc:512:replace_alu$177.CO[2]_new"
- note added: "$abc$2582$auto$alumacc.cc:512:replace_alu$177.CO[4]_new"
- note added: "$abc$2582$auto$alumacc.cc:512:replace_alu$180.CO[2]_new_inv"
- note added: "$abc$2582$auto$alumacc.cc:512:replace_alu$180.CO[4]_new_inv"
- note added: "$abc$2582$auto$alumacc.cc:512:replace_alu$183.CO[2]_new_inv"
- note added: "$abc$2582$auto$alumacc.cc:512:replace_alu$183.CO[5]_new_inv"
- note added: "$abc$2582$auto$alumacc.cc:512:replace_alu$183.CO[8]_new_inv"
- note added: "$abc$2582$auto$opt_dff.cc:272:make_patterns_logic$117_new"
- note added: "$abc$2582$auto$opt_dff.cc:272:make_patterns_logic$128_new"
- note added: "$abc$2582$auto$rtlil.cc:3584:NotGate$2363_new_inv"
- note added: "$abc$2582$auto$rtlil.cc:3584:NotGate$2379_new"
- note added: "$abc$2582$auto$simplemap.cc:148:simplemap_reduce$409[0]_new_inv"
- note added: "$abc$2582$auto$simplemap.cc:148:simplemap_reduce$413[0]_new_inv"
- note added: "$abc$2582$auto$simplemap.cc:148:simplemap_reduce$413[1]_new_inv"
- note added: "$abc$2582$auto$simplemap.cc:189:logic_reduce$333[1]_new_inv"
- note added: "$abc$2582$auto$simplemap.cc:189:logic_reduce$339[0]_new_inv"
- note added: "$abc$2582$auto$simplemap.cc:189:logic_reduce$339[1]_new_inv"
- note added: "$abc$2582$auto$simplemap.cc:189:logic_reduce$342_new_inv"
- note added: "$abc$2582$auto$simplemap.cc:189:logic_reduce$388_new_inv"
- note added: "$abc$2582$new_n103"
- note added: "$abc$2582$new_n112"
- note added: "$abc$2582$new_n117"
- note added: "$abc$2582$new_n121"
- note added: "$abc$2582$new_n125"
- note added: "$abc$2582$new_n128"
- note added: "$abc$2582$new_n129"
- note added: "$abc$2582$new_n130"
- note added: "$abc$2582$new_n131"
- note added: "$abc$2582$new_n132"
- note added: "$abc$2582$new_n133"
- note added: "$abc$2582$new_n136"
- note added: "$abc$2582$new_n139"
- note added: "$abc$2582$new_n141"
- note added: "$abc$2582$new_n143"
- note added: "$abc$2582$new_n145"
- note added: "$abc$2582$new_n148"
- note added: "$abc$2582$new_n150"
- note added: "$abc$2582$new_n152"
- note added: "$abc$2582$new_n155"
- note added: "$abc$2582$new_n158"
- note added: "$abc$2582$new_n161"
- note added: "$abc$2582$new_n164"
- note added: "$abc$2582$new_n75"
- note added: "$abc$2582$new_n76"
- note added: "$abc$2582$new_n86"
- note added: "$abc$2582$new_n87"
- note added: "$abc$2582$new_n92"
- note added: "$abc$2582$new_n93"
- note added: "$abc$2582$new_n96"
- note added: "$abc$2582$new_n97"
- note added: "$abc$2582$sol._25[2]_new_inv"
- note added: "$abc$2582$sol._25[3]_new_inv"
- note added: "$abc$2582$sol._25[4]_new_inv"
- note added: "$abc$2582$sol._27[5]_new_inv"
- note added: "$abc$2582$sol._27[6]_new_inv"
- note added: "$abc$2582$sol._31[6]_new_inv"
- note added: "$abc$2582$sol._33[4]_new"
- note added: "$abc$2582$sol._34[2]_new_inv"
- note added: "$abc$2582$sol._34[3]_new_inv"
- note added: "$abc$2582$sol._34[6]_new_inv"
- note added: "$abc$2582$sol._39[2]_new_inv"
- note added: "$abc$2582$sol._39[5]_new_inv"
- note added: "$abc$2582$sol._39[7]_new_inv"
- note added: "$auto$ff.cc:792:flip_bits$2361"
- note added: "$auto$ff.cc:792:flip_bits$2371"
- note added: "$auto$ff.cc:792:flip_bits$2377"
- note added: "SPECIAL_GND_NET"
- note added: "sol._15[0]"
- note added: "sol._15[1]"
- note added: "sol._15[2]"
- note added: "sol._15[3]"
- note added: "sol._15[4]"
- note added: "sol._15[5]"
- note added: "sol._15[6]"
- note added: "sol._15[7]"
- note added: "sol._15[8]"
- note added: "sol._15[9]"
- note added: "sol._20[0]"
- note added: "sol._20[2]"
- note added: "sol._20[3]"
- note added: "sol._20[6]"
- note added: "sol._21"
- note added: "step_count_0"
- note added: "step_count_1"
- note added: "step_count_2"
- note added: "step_count_3"
- note added: "step_count_4"
- note added: "step_count_5"
- note added: "step_count_6"
- note added: "step_count_7"
- note added: "step_count_8"
- note added: "step_count_9"
- note added: "step_direction"
- note added: "valid"
- note added: "zero_count_0"
- note added: "zero_count_1"
- note added: "zero_count_10"
- note added: "zero_count_2"
- note added: "zero_count_3"
- note added: "zero_count_4"
- note added: "zero_count_5"
- note added: "zero_count_6"
- note added: "zero_count_7"
- note added: "zero_count_8"
- note added: "zero_count_9"
- note removed: "The idea is that this sheet will be autogenerated, pointing to the global labels from the main sheet"
